File: hardware/raspberrypi-led-hat/raspberrypi-led-hat-2.sch (KiCad schematic (older format))
At the start: 8 parts, among them J1 Barrel_Jack, J2 Conn_01x03_Male, P1 Conn_02x20_Odd_Even, U1 BOB-12009

Commit message: Remade hat kicad and added readme
Parts:
- removed J2: Conn_01x03_Male, BOB-120009 Level Converter:Molex-0901362203, symbol Connector:Conn_01x03_Male
- added J2: Conn_02x02_Counter_Clockwise, footprints:430450400, symbol Connector_Generic:Conn_02x02_Counter_Clockwise
- added R1: R, Resistor_THT:R_Axial_DIN0204_L3.6mm_D1.6mm_P2.54mm_Vertical, symbol Device:R
- added SW1: SW_Push, Button_Switch_THT:SW_PUSH_6mm, symbol Switch:SW_Push
- MK1, MK2, MK3, MK4: symbol raspberrypi-led-hat-rescue:Mounting_Hole-Mechanical-raspberrypi-led-hat-rescue -> raspberrypi-led-hat-2-rescue:Mounting_Hole-Mechanical
- U1: footprint CONV_BOB-12009 -> BOB-120009 Level Converter:CONV_BOB-12009
Connections:
- net labels removed: LED_GROUND, LED_POWER
- wire segments 72 -> 57
Changed lines of the file:
@@
 Comment4 ""
 $EndDescr
-$Comp
-L power:+5V #PWR01
-U 1 1 580C1B61
-P 3100 950
-F 0 "#PWR01" H 3100 800 50  0001 C CNN
-F 1 "+5V" H 3100 1090 50  0000 C CNN
-F 2 "" H 3100 950 50  0000 C CNN
-F 3 "" H 3100 950 50  0000 C CNN
-	1    3100 950
-	1    0    0    -1
-$EndComp
 Wire Wire Line
 	3100 950  3100 1100
@@
 	2900 2900 3950 2900
 Wire Wire Line
+	2900 2300 3950 2300
+Wire Wire Line
 	2900 2400 3950 2400
 Wire Wire Line
 	2900 2100 3950 2100
 Wire Wire Line
+	2900 2200 3950 2200
+Wire Wire Line
 	2900 1800 3950 1800
 Wire Wire Line
@@
 Wire Wire Line
 	2900 1500 3950 1500
+Wire Wire Line
+	2900 1600 3950 1600
 Wire Wire Line
 	2900 1400 3950 1400
@@
 Text Label 3950 2400 2    50   ~ 0
 ID_SC
+Text Label 3950 2300 2    50   ~ 0
+GPIO7(SPI1_CE_N)
+Text Label 3950 2200 2    50   ~ 0
+GPIO8(SPI0_CE_N)
 Text Label 3950 2100 2    50   ~ 0
 GPIO25(GEN6)
@@
 ID_SD and ID_SC PINS:\nThese pins are reserved for HAT ID EEPROM.\n\nAt boot time this I2C interface will be\ninterrogated to look for an EEPROM\nthat identifes the attached board and\nallows automagic setup of the GPIOs\n(and optionally, Linux drivers).\n\nDO NOT USE these pins for anything other\nthan attaching an I2C ID EEPROM. Leave\nunconnected if ID EEPROM not required.
 $Comp
-L raspberrypi-led-hat-rescue:Mounting_Hole-Mechanical-raspberrypi-led-hat-rescue MK1
+L raspberrypi-led-hat-2-rescue:Mounting_Hole-Mechanical MK1
 U 1 1 5834FB2E
 P 3000 7200
@@
 $EndComp
 $Comp
-L raspberrypi-led-hat-rescue:Mounting_Hole-Mechanical-raspberrypi-led-hat-rescue MK3
+L raspberrypi-led-hat-2-rescue:Mounting_Hole-Mechanical MK3
 U 1 1 5834FBEF
 P 3450 7200
@@
 $EndComp
 $Comp
-L raspberrypi-led-hat-rescue:Mounting_Hole-Mechanical-raspberrypi-led-hat-rescue MK2
+L raspberrypi-led-hat-2-rescue:Mounting_Hole-Mechanical MK2
 U 1 1 5834FC19
 P 3000 7400
@@
 $EndComp
 $Comp
-L raspberrypi-led-hat-rescue:Mounting_Hole-Mechanical-raspberrypi-led-hat-rescue MK4
+L raspberrypi-led-hat-2-rescue:Mounting_Hole-Mechanical MK4
 U 1 1 5834FC4F
 P 3450 7400
@@
 $Comp
 L BOB-12009:BOB-12009 U1
-U 1 1 60A2181B
-P 2650 4550
-F 0 "U1" H 2650 5117 50  0000 C CNN
-F 1 "BOB-12009" H 2650 5026 50  0000 C CNN
-F 2 "CONV_BOB-12009" H 2650 4550 50  0001 L BNN
-F 3 "" H 2650 4550 50  0001 L BNN
-F 4 "SparkFun Electronics" H 2650 4550 50  0001 L BNN "MANUFACTURER"
-F 5 "N/A" H 2650 4550 50  0001 L BNN "MAXIMUM_PACKAGE_HEIGHT"
-F 6 "Manufacturer Recommendations" H 2650 4550 50  0001 L BNN "STANDARD"
-F 7 "01" H 2650 4550 50  0001 L BNN "PARTREV"
-	1    2650 4550
-	1    0    0    -1
-$EndComp
-Wire Wire Line
-	2000 4450 1950 4450
-Connection ~ 1950 4450
-Wire Wire Line
-	1950 4450 1850 4450
-Wire Wire Line
-	2200 1100 1000 1100
-Wire Wire Line
-	1000 1100 1000 4250
-Wire Wire Line
-	1000 4250 1950 4250
-Wire Wire Line
-	3350 4950 3700 4950
-Wire Wire Line
-	3700 4950 3700 4650
-Wire Wire Line
-	3700 3150 3000 3150
-Connection ~ 3000 3150
-Wire Wire Line
-	3350 4250 3550 4250
-Wire Wire Line
-	3700 4950 3750 4950
-Connection ~ 3700 4950
-Connection ~ 3550 4550
-Connection ~ 3700 4650
-Wire Wire Line
-	3700 4650 3700 3150
-Text Label 5500 4450 0    50   ~ 0
+U 1 1 60C05AD4
+P 1900 4550
+F 0 "U1" H 1900 5117 50  0000 C CNN
+F 1 "BOB-12009" H 1900 5026 50  0000 C CNN
+F 2 "BOB-120009 Level Converter:CONV_BOB-12009" H 1900 4550 50  0001 L BNN
+F 3 "" H 1900 4550 50  0001 L BNN
+F 4 "SparkFun Electronics" H 1900 4550 50  0001 L BNN "MANUFACTURER"
+F 5 "N/A" H 1900 4550 50  0001 L BNN "MAXIMUM_PACKAGE_HEIGHT"
+F 6 "Manufacturer Recommendations" H 1900 4550 50  0001 L BNN "STANDARD"
+F 7 "01" H 1900 4550 50  0001 L BNN "PARTREV"
+	1    1900 4550
+	1    0    0    -1
+$EndComp
+Wire Wire Line
+	550  4450 1200 4450
+$Comp
+L power:+3.3V #PWR0101
+U 1 1 60C20272
+P 1200 4250
+F 0 "#PWR0101" H 1200 4100 50  0001 C CNN
+F 1 "+3.3V" V 1215 4378 50  0000 L CNN
+F 2 "" H 1200 4250 50  0001 C CNN
+F 3 "" H 1200 4250 50  0001 C CNN
+	1    1200 4250
+	0    -1   -1   0
+$EndComp
+Text Label 550  4450 0    30   ~ 0
+GPIO18(GEN1)(PWM0)
+$Comp
+L Connector:Barrel_Jack J1
+U 1 1 60C2244A
+P 1600 5400
+F 0 "J1" H 1657 5725 50  0000 C CNN
+F 1 "Barrel_Jack" H 1657 5634 50  0000 C CNN
+F 2 "Connector_BarrelJack:BarrelJack_CUI_PJ-063AH_Horizontal" H 1650 5360 50  0001 C CNN
+F 3 "~" H 1650 5360 50  0001 C CNN
+	1    1600 5400
+	1    0    0    -1
+$EndComp
+$Comp
+L power:GND #PWR0102
+U 1 1 60C23361
+P 1900 5500
+F 0 "#PWR0102" H 1900 5250 50  0001 C CNN
+F 1 "GND" V 1905 5372 50  0000 R CNN
+F 2 "" H 1900 5500 50  0001 C CNN
+F 3 "" H 1900 5500 50  0001 C CNN
+	1    1900 5500
+	0    -1   -1   0
+$EndComp
+$Comp
+L power:+5V #PWR0103
+U 1 1 60C23BC2
+P 1900 5300
+F 0 "#PWR0103" H 1900 5150 50  0001 C CNN
+F 1 "+5V" V 1915 5428 50  0000 L CNN
+F 2 "" H 1900 5300 50  0001 C CNN
+F 3 "" H 1900 5300 50  0001 C CNN
+	1    1900 5300
+	0    1    1    0
+$EndComp
+$Comp
+L power:GND #PWR0104
+U 1 1 60C2418B
+P 2600 4950
+F 0 "#PWR0104" H 2600 4700 50  0001 C CNN
+F 1 "GND" V 2605 4822 50  0000 R CNN
+F 2 "" H 2600 4950 50  0001 C CNN
+F 3 "" H 2600 4950 50  0001 C CNN
+	1    2600 4950
+	0    -1   -1   0
+$EndComp
+Text Label 2200 6050 0    30   ~ 0
 LED_DATA
-Text Label 5500 4550 0    50   ~ 0
-LED_POWER
-Text Label 5500 4650 0    50   ~ 0
-LED_GROUND
-$Comp
-L Connector:Barrel_Jack J1
-U 1 1 609CFBCC
-P 3650 6500
-F 0 "J1" V 3753 6320 50  0000 R CNN
-F 1 "Barrel_Jack" V 3662 6320 50  0000 R CNN
-F 2 "Connector_BarrelJack:BarrelJack_CUI_PJ-063AH_Horizontal" H 3700 6460 50  0001 C CNN
-F 3 "~" H 3700 6460 50  0001 C CNN
-	1    3650 6500
-	0    -1   -1   0
-$EndComp
-Wire Wire Line
-	3550 4250 3550 4550
-Wire Wire Line
-	3750 4950 3750 6200
-Wire Wire Line
-	3550 4550 3550 6200
-Wire Wire Line
-	3350 4450 6100 4450
-Wire Wire Line
-	3550 4550 6100 4550
-Wire Wire Line
-	3700 4650 6100 4650
-$Comp
-L Connector:Conn_01x03_Male J2
-U 1 1 609FFB72
-P 6300 4550
-F 0 "J2" H 6272 4482 50  0000 R CNN
-F 1 "Conn_01x03_Male" H 6272 4573 50  0000 R CNN
-F 2 "BOB-120009 Level Converter:Molex-0901362203" H 6300 4550 50  0001 C CNN
-F 3 "~" H 6300 4550 50  0001 C CNN
-	1    6300 4550
-	-1   0    0    1
-$EndComp
-Wire Wire Line
-	2900 2200 3950 2200
-Text Label 3950 2200 2    50   ~ 0
-GPIO8(SPI0_CE_N)
-Text Label 3950 2300 2    50   ~ 0
-GPIO7(SPI1_CE_N)
-Wire Wire Line
-	2900 2300 3950 2300
-Wire Wire Line
-	1850 4450 1850 3850
-Wire Wire Line
-	1850 3850 4050 3850
-Wire Wire Line
-	4050 3850 4050 1600
-Wire Wire Line
-	2900 1600 4050 1600
+$Comp
+L power:+5V #PWR0106
+U 1 1 60C32C17
+P 1700 6050
+F 0 "#PWR0106" H 1700 5900 50  0001 C CNN
+F 1 "+5V" V 1715 6178 50  0000 L CNN
+F 2 "" H 1700 6050 50  0001 C CNN
+F 3 "" H 1700 6050 50  0001 C CNN
+	1    1700 6050
+	0    -1   -1   0
+$EndComp
+$Comp
+L power:+5V #PWR0107
+U 1 1 60C353E9
+P 2600 4250
+F 0 "#PWR0107" H 2600 4100 50  0001 C CNN
+F 1 "+5V" V 2615 4378 50  0000 L CNN
+F 2 "" H 2600 4250 50  0001 C CNN
+F 3 "" H 2600 4250 50  0001 C CNN
+	1    2600 4250
+	0    1    1    0
+$EndComp
+Wire Wire Line
+	2600 4450 2800 4450
+Text Label 2600 4450 0    30   ~ 0
+LED_DATA
+Wire Wire Line
+	2200 6050 2400 6050
+Text Label 2200 6150 0    30   ~ 0
+LED_DATA
+Wire Wire Line
+	2200 6150 2400 6150
+$Comp
+L Switch:SW_Push SW1
+U 1 1 60C6047C
+P 3050 5500
+F 0 "SW1" H 3050 5785 50  0000 C CNN
+F 1 "SW_Push" H 3050 5694 50  0000 C CNN
+F 2 "Button_Switch_THT:SW_PUSH_6mm" H 3050 5700 50  0001 C CNN
+F 3 "~" H 3050 5700 50  0001 C CNN
+	1    3050 5500
+	1    0    0    -1
+$EndComp
+$Comp
+L power:+3.3V #PWR0108
+U 1 1 60C6B277
+P 2850 5500
+F 0 "#PWR0108" H 2850 5350 50  0001 C CNN
+F 1 "+3.3V" V 2865 5628 50  0000 L CNN
+F 2 "" H 2850 5500 50  0001 C CNN
+F 3 "" H 2850 5500 50  0001 C CNN
+	1    2850 5500
+	0    -1   -1   0
+$EndComp
+$Comp
+L Device:R R1
+U 1 1 60C6D8BB
+P 3400 5500
+F 0 "R1" V 3607 5500 50  0000 C CNN
+F 1 "R" V 3516 5500 50  0000 C CNN
+F 2 "Resistor_THT:R_Axial_DIN0204_L3.6mm_D1.6mm_P2.54mm_Vertical" V 3330 5500 50  0001 C CNN
+F 3 "~" H 3400 5500 50  0001 C CNN
+	1    3400 5500
+	0    -1   -1   0
+$EndComp
+Wire Wire Line
+	3550 5500 3800 5500
+Text Label 3800 5500 0    30   ~ 0
+GPIO15(RXD0)
+$Comp
+L Connector_Generic:Conn_02x02_Counter_Clockwise J2
+U 1 1 60C3EE0D
+P 1900 6050
+F 0 "J2" H 1950 6267 50  0000 C CNN
+F 1 "Conn_02x02_Counter_Clockwise" H 1950 6176 50  0000 C CNN
+F 2 "footprints:430450400" H 1900 6050 50  0001 C CNN
+F 3 "~" H 1900 6050 50  0001 C CNN
+	1    1900 6050
+	1    0    0    -1
+$EndComp
+$Comp
+L power:GND #PWR0105
+U 1 1 60C326FE
+P 1700 6150
+F 0 "#PWR0105" H 1700 5900 50  0001 C CNN
+F 1 "GND" V 1705 6022 50  0000 R CNN
+F 2 "" H 1700 6150 50  0001 C CNN
+F 3 "" H 1700 6150 50  0001 C CNN
+	1    1700 6150
+	0    1    1    0
+$EndComp
 $EndSCHEMATC
